File: ti84_usbc.kicad_sch (KiCad schematic)
At the start: 6 parts, among them J1 USB_C_Receptacle_USB2.0, J2 USB_OTG, U1 TUSB320

Commit message: Add files via upload
Parts:
- U1: footprint Package_DFN_QFN:Texas_X2QFN-12_1.6x1.6mm_P0.4mm -> ti84_mini_usb:IC_TUSB320IRWBR
Changed lines of the file:
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@@
       (effects (font (size 1.27 1.27)) (justify left))
     )
-    (property "Footprint" "Package_DFN_QFN:Texas_X2QFN-12_1.6x1.6mm_P0.4mm" (at 149.86 133.35 0)
+    (property "Footprint" "ti84_mini_usb:IC_TUSB320IRWBR" (at 149.86 133.35 0)
       (effects (font (size 1.27 1.27)) hide)
     )
